Commit message: created launch files

File: kendama_description/urdf/kendama.urdf.xacro (robot description, xacro)
@@ -1,4 +1,4 @@
 <robot name="kendama" xmlns:xacro="http://www.ros.org/wiki/xacro">
-  <xacro:include filename="(find kendama_description)/urdf/kendama.xacro"/>
-  <xacro:kendama/>
+  <xacro:include filename="$(find kendama_description)/urdf/kendama.xacro"/>
+  <xacro:kendama parent="base_link"/>
 </robot>

File: kendama_description/urdf/kendama.xacro (robot description, xacro)
@@ -1,7 +1,7 @@
-<robot name="hc_sr04" xmlns:xacro="http://www.ros.org/wiki/xacro">
-  <xacro:macro name="kendama">
+<robot name="kendama" xmlns:xacro="http://www.ros.org/wiki/xacro">
+  <xacro:macro name="kendama" params="parent">
     <link name="ken_link">
       <visual>
-	<origin xyz="0 0 0" rpy="0 0 0"/>
+	<origin xyz="0 0 0" rpy="1.5708 0 0"/>
 	<geometry>
 	  <mesh filename = "file::///$(find kendama_description)/meshes/ken.STL"

Commit message: launch files working; ur5 and kendama show up in rviz

File: kendama_description/urdf/kendama.urdf.xacro (robot description, xacro)
@@ -1,4 +1,12 @@
-<robot name="kendama" xmlns:xacro="http://www.ros.org/wiki/xacro">
+<robot name="kendama_on_ur5" xmlns:xacro="http://www.ros.org/wiki/xacro">
+  <xacro:include filename="$(find ur_description)/urdf/ur5.urdf.xacro"/>
   <xacro:include filename="$(find kendama_description)/urdf/kendama.xacro"/>
+  <xacro:ur5_robot prefix="" joint_limited="true"/>
   <xacro:kendama parent="tool0"/>
+  <link name="world"/>
+  <joint name="world_joint" type="fixed">
+    <parent link="world"/>
+    <child link="base_link"/>
+    <origin xyz="0.0 0.0 0.0" rpy="0.0 0.0 0.0"/>
+  </joint>
 </robot>

File: kendama_description/urdf/kendama.xacro (robot description, xacro)
@@ -5,5 +5,5 @@
 	<origin xyz="0 0 0" rpy="1.5708 0 0"/>
 	<geometry>
-	  <mesh filename = "file::///$(find kendama_description)/meshes/ken.STL"
+	  <mesh filename = "file::///$(find kendama_description)/meshes/visual/ken.STL"
 		scale = "0.001 0.001 0.001"/>
 	</geometry>
@@ -14,5 +14,5 @@
       <collision>
 	<geometry>
-	  <mesh filename = "file::///$(find kendama_description)/meshes/ken_simple.STL"
+	  <mesh filename = "file::///$(find kendama_description)/meshes/collision/ken_simple.STL"
 		scale = "0.001 0.001 0.001"/>
 	</geometry>

Commit message: copied/modified existing ur5 description and launch files to add kendama

File: kendama_description/urdf/kendama.urdf.xacro (robot description, xacro)
@@ -1,6 +1,6 @@
 <robot name="kendama_on_ur5" xmlns:xacro="http://www.ros.org/wiki/xacro">
-  <xacro:include filename="$(find ur_description)/urdf/ur5.urdf.xacro"/>
+<!--  <xacro:include filename="$(find ur_description)/urdf/ur5.urdf.xacro"/> -->
   <xacro:include filename="$(find kendama_description)/urdf/kendama.xacro"/>
-  <xacro:ur5_robot prefix="" joint_limited="true"/>
+<!--  <xacro:ur5_robot prefix="" joint_limited="true"/> -->
   <xacro:kendama parent="tool0"/>
   <link name="world"/>

File: kendama_description/urdf/kendama.xacro (robot description, xacro)
@@ -3,13 +3,15 @@
     <link name="ken_mount_link">
       <visual>
-	<origin xyz="0 0 0.006" rpy="0 0 0"/>
+	<origin xyz="0 0 0.006" rpy="-1.5708 0 0.7854"/>
 	<geometry>
-	  <cylinder radius="0.0375" length="0.012"/>
+	  <mesh filename = "file::///$(find kendama_description)/meshes/visual/kendama_mount.STL"
+		scale = "0.001 0.001 0.001"/>
 	</geometry>
-	<material name="acrylic">
+	<material name="blue_acrylic">
 	  <color rgba="0 0 0.75 0.5"/>
 	</material>
       </visual>
       <collision>
+	<origin xyz="0 0 0.006" rpy="0 0 0"/>
 	<geometry>
 	  <cylinder radius="0.0375" length="0.012"/>
@@ -29,5 +31,5 @@
 	</geometry>
 	<material name = "wood">
-	  <color rgba="0.59 0.44 0.20 0.5"/>
+	  <color rgba="0.59 0.44 0.20 1"/>
 	</material>
       </visual>
