Commit message: added the kendama_mount to kendama_description and updated STLs

File: kendama_description/urdf/kendama.xacro (robot description, xacro)
@@ -1,7 +1,27 @@
 <robot name="kendama" xmlns:xacro="http://www.ros.org/wiki/xacro">
   <xacro:macro name="kendama" params="parent">
+    <link name="ken_mount_link">
+      <visual>
+	<origin xyz="0 0 0.006" rpy="0 0 0"/>
+	<geometry>
+	  <cylinder radius="0.0375" length="0.012"/>
+	</geometry>
+	<material name="acrylic">
+	  <color rgba="0 0 0.75 0.5"/>
+	</material>
+      </visual>
+      <collision>
+	<geometry>
+	  <cylinder radius="0.0375" length="0.012"/>
+	</geometry>
+      </collision>
+    </link>
+    <joint name="ken_mount_joint" type="fixed">
+      <parent link="${parent}"/>
+      <child link="ken_mount_link"/>
+    </joint>
     <link name="ken_link">
       <visual>
-	<origin xyz="0 0 0" rpy="1.5708 0 0"/>
+	<origin xyz="0 0 0.006" rpy="1.5708 0 0"/>
 	<geometry>
 	  <mesh filename = "file::///$(find kendama_description)/meshes/visual/ken.STL"
@@ -20,5 +40,5 @@
     </link>
     <joint name="ken_joint" type="fixed">
-      <parent link="${parent}"/>
+      <parent link="ken_mount_link"/>
       <child link="ken_link"/>
     </joint>

Commit message: added semi-random inertial info to kendama xacro

File: kendama_description/urdf/kendama.xacro (robot description, xacro)
@@ -18,4 +18,9 @@
 	</geometry>
       </collision>
+      <inertial>
+	<origin xyz="0 0 0.006" rpy="0 0 0"/>
+	<mass value="0.05"/>
+	<inertia ixx="0" ixy="0" ixz="0" iyy="0" iyz="0" izz="0"/>
+      </inertial>
     </link>
     <joint name="ken_mount_joint" type="fixed">
@@ -40,4 +45,9 @@
 	</geometry>
       </collision>
+      <inertial>
+	<origin xyz="0 0 0.006" rpy="1.5708 0 0"/>
+	<mass value="0.05"/>
+	<inertia ixx="0" ixy="0" ixz="0" iyy="0" iyz="0" izz="0"/>
+      </inertial>
     </link>
     <joint name="ken_joint" type="fixed">

Commit message: added kendama stl stuff

File: kendama_description/urdf/kendama.xacro (robot description, xacro)
@@ -2,56 +2,65 @@
   <xacro:macro name="kendama" params="parent">
     <link name="ken_mount_link">
-      <visual>
-	<origin xyz="0 0 0.006" rpy="-1.5708 0 0.7854"/>
-	<geometry>
-	  <mesh filename = "file::///$(find kendama_description)/meshes/visual/kendama_mount.STL"
-		scale = "0.001 0.001 0.001"/>
-	</geometry>
-	<material name="blue_acrylic">
-	  <color rgba="0 0 0.75 0.5"/>
-	</material>
-      </visual>
-      <collision>
-	<origin xyz="0 0 0.006" rpy="0 0 0"/>
-	<geometry>
-	  <cylinder radius="0.0375" length="0.012"/>
-	</geometry>
-      </collision>
-      <inertial>
-	<origin xyz="0 0 0.006" rpy="0 0 0"/>
-	<mass value="0.05"/>
-	<inertia ixx="0" ixy="0" ixz="0" iyy="0" iyz="0" izz="0"/>
-      </inertial>
+    	<visual>
+			<origin xyz="0.0 0.0 0.0" rpy="0.0 0.0 0.0"/>
+			<geometry>
+				<mesh filename = "file://$(find kendama_description)/meshes/visual/kendama_mount.STL"
+					scale="0.001 0.001 0.001"/>
+			</geometry>
+			<material name="blue_acrylic">
+				<color rgba="0 0 0.75 0.5"/>
+			</material>
+      	</visual>
+      	<collision>
+			<origin xyz="0.0 0.0 0.0" rpy="0.0 0.0 0.0"/>
+			<geometry>
+				<cylinder radius="0.0375" length="0.012"/>
+			</geometry>
+      	</collision>
+      	<inertial>
+			<origin xyz="0.0 0.0 0.0" rpy="0.0 0.0 0.0"/>
+			<mass value="0.05"/>
+			<inertia ixx="0.001" ixy="0" ixz="0" iyy="0.001" iyz="0" izz="0.001"/>
+      	</inertial>
     </link>
-    <joint name="ken_mount_joint" type="fixed">
-      <parent link="${parent}"/>
-      <child link="ken_mount_link"/>
+    <link name="ken_link">
+    	<visual>
+			<origin xyz="0.0 0.0 0.0" rpy="0.0 0.0 0.0"/>
+			<geometry>
+				<mesh filename="file://$(find kendama_description)/meshes/visual/ken.STL"
+					scale="0.001 0.001 0.001"/>
+			</geometry>
+			<material name = "wood">
+				<color rgba="0.59 0.44 0.20 1"/>
+			</material>
+      	</visual>
+		<collision>
+			<origin xyz="0.0 0.0 0.0" rpy="0.0 0.0 0.0"/>
+			<geometry>
+				<mesh filename="file://$(find kendama_description)/meshes/collision/ken.STL"
+					scale="0.001 0.001 0.001"/>
+			</geometry>
+		</collision>
+		<inertial>
+			<origin xyz="0.0 0.0 0.0" rpy="0.0 0.0 0.0"/>
+			<mass value="0.05"/>
+			<inertia ixx="0.001" ixy="0" ixz="0" iyy="0.001" iyz="0" izz="0.001"/>
+		</inertial>
+    </link>
+	<link name="cup_link"/>
+	<joint name="ken_mount_joint" type="fixed">
+      	<parent link="${parent}"/>
+      	<child link="ken_mount_link"/>
+	  	<origin xyz="0 0 0.006" rpy="-1.5708 0 0.7854"/>
     </joint>
-    <link name="ken_link">
-      <visual>
-	<origin xyz="0 0 0.006" rpy="1.5708 0 0"/>
-	<geometry>
-	  <mesh filename = "file::///$(find kendama_description)/meshes/visual/ken.STL"
-		scale = "0.001 0.001 0.001"/>
-	</geometry>
-	<material name = "wood">
-	  <color rgba="0.59 0.44 0.20 1"/>
-	</material>
-      </visual>
-      <collision>
-	<geometry>
-	  <mesh filename = "file::///$(find kendama_description)/meshes/collision/ken_simple.STL"
-		scale = "0.001 0.001 0.001"/>
-	</geometry>
-      </collision>
-      <inertial>
-	<origin xyz="0 0 0.006" rpy="1.5708 0 0"/>
-	<mass value="0.05"/>
-	<inertia ixx="0" ixy="0" ixz="0" iyy="0" iyz="0" izz="0"/>
-      </inertial>
-    </link>
     <joint name="ken_joint" type="fixed">
       <parent link="ken_mount_link"/>
       <child link="ken_link"/>
+	  <origin xyz="0 0 0" rpy="3.1415 2.3561 0"/>
+    </joint>
+	<joint name="cup_joint" type="fixed">
+      <parent link="ken_link"/>
+      <child link="cup_link"/>
+	  <origin xyz="-0.02637 0.106 0.0" rpy="0 -1.5708 0"/>
     </joint>
   </xacro:macro>

Commit message: Started to create sim/hardware launch packages

File: kendama_description/urdf/kendama.xacro (robot description, xacro)
@@ -38,5 +38,5 @@
 			<origin xyz="0.0 0.0 0.0" rpy="0.0 0.0 0.0"/>
 			<geometry>
-				<mesh filename="file://$(find kendama_description)/meshes/collision/ken.STL"
+				<mesh filename="file://$(find kendama_description)/meshes/collision/ken_collision.STL"
 					scale="0.001 0.001 0.001"/>
 			</geometry>
